Commit message: Human model simulation nominally working

File: drake/examples/human_model/models/simplified_human_model.urdf (robot description, URDF)
Before this commit: robot human, 68 links, 67 joints
Joints:
- joint jC1Head_X: type revolute -> continuous
- joint jC1Head_Y: type revolute -> continuous
- joint jC1Head_Z: type revolute -> continuous
- joint jL1T12_X: type revolute -> continuous
- joint jL1T12_Y: type revolute -> continuous
- joint jL1T12_Z: type revolute -> continuous
- joint jL4L3_X: type revolute -> continuous
- joint jL4L3_Y: type revolute -> continuous
- joint jL4L3_Z: type revolute -> continuous
- joint jL5S1_X: type revolute -> continuous
- joint jL5S1_Y: type revolute -> continuous
- joint jL5S1_Z: type revolute -> continuous
- joint jLeftAnkle_X: type revolute -> continuous
- joint jLeftAnkle_Y: type revolute -> continuous
- joint jLeftAnkle_Z: type revolute -> continuous
- joint jLeftBallFoot_X: type revolute -> continuous
- joint jLeftBallFoot_Y: type revolute -> continuous
- joint jLeftBallFoot_Z: type revolute -> continuous
- joint jLeftC7Shoulder_X: type revolute -> continuous
- joint jLeftC7Shoulder_Y: type revolute -> continuous
- joint jLeftC7Shoulder_Z: type revolute -> continuous
- joint jLeftElbow_X: type revolute -> continuous
- joint jLeftElbow_Y: type revolute -> continuous
- joint jLeftElbow_Z: type revolute -> continuous
- joint jLeftHip_X: type revolute -> continuous
- joint jLeftHip_Y: type revolute -> continuous
- joint jLeftHip_Z: type revolute -> continuous
- joint jLeftKnee_X: type revolute -> continuous
- joint jLeftKnee_Y: type revolute -> continuous
- joint jLeftKnee_Z: type revolute -> continuous
- joint jLeftShoulder_X: type revolute -> continuous
- joint jLeftShoulder_Y: type revolute -> continuous
- joint jLeftShoulder_Z: type revolute -> continuous
- joint jLeftWrist_X: type revolute -> continuous
- joint jLeftWrist_Y: type revolute -> continuous
- joint jLeftWrist_Z: type revolute -> continuous
- joint jRightAnkle_X: type revolute -> continuous
- joint jRightAnkle_Y: type revolute -> continuous
- joint jRightAnkle_Z: type revolute -> continuous
- joint jRightBallFoot_X: type revolute -> continuous
- joint jRightBallFoot_Y: type revolute -> continuous
- joint jRightBallFoot_Z: type revolute -> continuous
- joint jRightC7Shoulder_X: type revolute -> continuous
- joint jRightC7Shoulder_Y: type revolute -> continuous
- joint jRightC7Shoulder_Z: type revolute -> continuous
- joint jRightElbow_X: type revolute -> continuous
- joint jRightElbow_Y: type revolute -> continuous
- joint jRightElbow_Z: type revolute -> continuous
- joint jRightHip_X: type revolute -> continuous
- joint jRightHip_Y: type revolute -> continuous
- joint jRightHip_Z: type revolute -> continuous
- joint jRightKnee_X: type revolute -> continuous
- joint jRightKnee_Y: type revolute -> continuous
- joint jRightKnee_Z: type revolute -> continuous
- joint jRightShoulder_X: type revolute -> continuous
- joint jRightShoulder_Y: type revolute -> continuous
- joint jRightShoulder_Z: type revolute -> continuous
- joint jRightWrist_X: type revolute -> continuous
- joint jRightWrist_Y: type revolute -> continuous
- joint jRightWrist_Z: type revolute -> continuous
- joint jT1C7_X: type revolute -> continuous
- joint jT1C7_Y: type revolute -> continuous
- joint jT1C7_Z: type revolute -> continuous
- joint jT9T8_X: type revolute -> continuous
- joint jT9T8_Y: type revolute -> continuous
- joint jT9T8_Z: type revolute -> continuous

Commit message: update human simulation model

File: drake/examples/human_model/models/simplified_human_model.urdf (robot description, URDF)
Before this commit: robot human, 68 links, 67 joints
Links:
- link Left Upper Leg: geometry collision cylinder length=0.442 radius=0.0806551326413; visual cylinder length=0.442 radius=0.0806551326413
- link Right Upper Leg: geometry collision cylinder length=0.442 radius=0.0806551326413; visual cylinder length=0.442 radius=0.0806551326413
